File: EB-STM32L412KB.kicad_pcb (KiCad board)
At the start: 2 copper layers, 20 x 49 mm, 25 parts, among them J1 USB_B_Micro, J2 STDC32, J3 Conn_01x13, J4 Conn_01x13, SW1 RESET_SW, U1 LXES11DAA2-135, U2 FT234XD, U3 STM32L412KBTx, Y1 32.768kHz

Commit message: 基盤V2.0
Parts:
- removed TP3, TP4: TestPoint, EB-STM32L412KB:TestPoint_THTPad_D1.6mm_Drill1.0mm
- added R3: 10k, EB-STM32L412KB:1608Metric, F.Cu at (4.50, 15.5)
- added SW2: SW_DPDT, EB-STM32L412KB:IS-2235-G, F.Cu at (0.00, 10.6)
- J3, J4: value Conn_01x13 -> Conn_01x14; footprint EB-STM32L412KB:PinHeader_13pin -> EB-STM32L412KB:PinHeader_14pin
- U3: footprint EB-STM32L412KB:LQFP-32_7x7mm_P0.8mm_FusionPCB -> EB-STM32L412KB:QFN-32-1EP_5x5mm_P0.5mm_EP3.3x3.3mm
- moved C5 3.35 mm to (-0.40, 14.4)
- moved C6 3.35 mm to (-2.60, 14.4)
- moved Y1 3.35 mm to (-1.50, 16.0)
- moved C3 3.23 mm to (3.00, 15.5)
- moved SW1 2.50 mm to (0.00, 31.0)
- moved U3 2.50 mm to (0.00, 22.5)
- moved C4 2.40 mm to (-4.30, 30.9)
Connections:
- net +3V3 renamed +3.3V
- J1 pad 4: (no net) -> unconnected-(J1-Pad4)
- J2 pad 1: (no net) -> unconnected-(J2-Pad1)
- J2 pad 10: (no net) -> unconnected-(J2-Pad10)
- J2 pad 13: (no net) -> unconnected-(J2-Pad13)
- J2 pad 14: (no net) -> unconnected-(J2-Pad14)
- J2 pad 2: (no net) -> unconnected-(J2-Pad2)
- J2 pad 8: (no net) -> unconnected-(J2-Pad8)
- J2 pad 9: (no net) -> unconnected-(J2-Pad9)
- J4 pad 10: PA11 -> PA15
- J4 pad 11: PA10 -> PA12
- J4 pad 12: PA9 -> PA11
- J4 pad 13: PA8 -> PA10
- J4 pad 5: PB5 -> PB7
- J4 pad 6: PB4 -> PB6
- J4 pad 7: PB3 -> PB5
- J4 pad 8: PA15 -> PB4
- J4 pad 9: PA12 -> PB3
- U1 pad 4: /DM -> USBDM
- U1 pad 5: /DP -> USBDP
- U2 pad 1: /DM -> FT_DM
- U2 pad 10: USART1_TX -> PB6
- U2 pad 11: (no net) -> unconnected-(U2-Pad11)
- U2 pad 12: /DP -> FT_DP
- U2 pad 7: USART1_RX -> PB7
- U2 pad 8: (no net) -> unconnected-(U2-Pad8)
- U3 pad 29: USART1_TX -> PB6
- U3 pad 30: USART1_RX -> PB7
Routing:
- net GND: track 236.7 -> 144.2 mm, vias 5 -> 2
- net USART1_TX: track 28.3 -> 0.00 mm, vias 2 -> 0
- net PB6: track 0.00 -> 23.8 mm, vias 0 -> 1
- net PB7: track 0.00 -> 21.1 mm, vias 0 -> 1
- net USART1_RX: track 20.2 -> 0.00 mm, vias 1 -> 0
- net PA12: track 10.7 -> 28.8 mm
- net PA11: track 10.8 -> 28.6 mm
- net NRST: track 54.6 -> 39.7 mm, vias 3 -> 2
- net USBDM: track 0.00 -> 14.0 mm, vias 0 -> 1
- net FT_DM: track 0.00 -> 12.1 mm, vias 0 -> 1
- net FT_DP: track 0.00 -> 12.0 mm, vias 0 -> 1
- net USBDP: track 0.00 -> 9.99 mm, vias 0 -> 1
- net /DM: track 8.61 -> 0.00 mm, vias 2 -> 0
- net PA8: track 15.7 -> 21.0 mm
- net PA0: track 11.6 -> 16.4 mm
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Other:
- board size 20 x 49 mm -> 20 x 51.5 mm
- net class Default removed
- board text added: "PB6"
- board text added: "PB7"
- board text removed: "Rx"
- board text removed: "Tx"
